File: kicad/nano_nrf/nano_nrf.sch (KiCad schematic (older format))
At the start: 3 parts, among them P1 Digital, P2 Analog, P3 CONN_02X04

Commit message: Leds
Parts:
- added D1, D2: LED, LEDs:LED-5MM, symbol LED
- added D3: LED_RCBG, LEDs:LED-RGB-5MM_Common_Cathode, symbol LED_RCBG
- added P4, P5: CONN_01X06, Socket_Strips:Socket_Strip_Straight_1x06, symbol CONN_01X06
- added R1, R2, R4, R5: 100R, Resistors_ThroughHole:Resistor_Horizontal_RM10mm, symbol R
- added R3: 180R, Resistors_ThroughHole:Resistor_Horizontal_RM10mm, symbol R
Connections:
- net labels added: 10(SS), 3, 5, 5V, 6, 9, A4(SDA), A5(SCL), LED_GREEN, LED_RED, RGB_BLUE, RGB_GREEN, RGB_RED
- net labels removed: +3.3V, +5V, 0(Rx), 1(Tx), 10(**/SS), 2, 3(**), 4, 5(**), 6(**), 9(**), A1, A2, A3, A4, A5, A6, A7, AREF, Reset, Vin
- wire segments 41 -> 45
- no-connect marks 1 -> 15
Other:
- note added: "Arduino Nano"
- note removed: "Shield for Arduino Nano"
- moved on the sheet: P3

Commit message: Nano on the bottom
Connections:
- net 11(MISO) renamed 11(MOSI)
- net 11(MOSI): now also P3.6 (P6); no longer P3.7 (P7)
- net 12(MOSI) renamed 12(MISO)
- net 12(MISO): now also P3.7 (P7); no longer P3.6 (P6)
Changed lines of the file:
@@
 Text Label 8550 2500 0    60   ~ 0
 10(SS)
-Text Label 10250 3975 0    60   ~ 0
-11(MISO)
 Text Label 8550 2700 0    60   ~ 0
-12(MOSI)
+12(MISO)
 Text Label 10750 2700 0    60   ~ 0
 13(SCK)
@@
 13(SCK)
 Text Label 8550 2600 0    60   ~ 0
-11(MISO)
-Text Label 9075 4075 0    60   ~ 0
-12(MOSI)
+11(MOSI)
 Text Label 9075 4175 0    60   ~ 0
 8
@@
 Text Label 6600 4350 0    60   ~ 0
 5V
-Text Label 8050 4150 0    60   ~ 0
-11(MISO)
-Text Label 8050 4250 0    60   ~ 0
-12(MOSI)
 Text Label 8050 4350 0    60   ~ 0
 13(SCK)
@@
 Wire Wire Line
 	9275 2400 8550 2400
+Text Label 8050 4250 0    60   ~ 0
+12(MISO)
+Text Label 8050 4150 0    60   ~ 0
+11(MOSI)
+Text Label 9075 4075 0    60   ~ 0
+11(MOSI)
+Text Label 10250 3975 0    60   ~ 0
+12(MISO)
 $EndSCHEMATC

Commit message: Swap SDA & SCL
Parts:
- added P10: CONN_01X02, Socket_Strips:Socket_Strip_Straight_1x02, symbol CONN_01X02
Connections:
- net 10(SS): now also P5.6 (P6); no longer P5.1 (P1)
- net 11(MOSI): now also P5.5 (P5); no longer P5.2 (P2)
- net 12(MISO): now also P5.4 (P4); no longer P5.3 (P3)
- net 13(SCK): now also P5.3 (P3); no longer P5.4 (P4)
- net 3V3: now also P4.2 (P2), P5.2 (P2); no longer P4.5 (P5), P5.5 (P5)
- net 5V: now also P10.2 (P2); no longer P4.4 (P4)
- net A0: now also P4.6 (P6); no longer P4.1 (P1)
- net A4(SDA): now also P4.4 (P4); no longer P4.2 (P2)
- net GND: now also P4.1 (P1), P5.1 (P1), P10.1 (P1); no longer P4.6 (P6), P5.6 (P6)
- net A1: now reaches P2.11 (P11)
- net A1: now also P4.5 (P5)
- no-connect marks 15 -> 14
Changed lines of the file:
@@
 F 3 "" H 7175 4300 50  0000 C CNN
 	1    7175 4300
-	1    0    0    -1
+	1    0    0    1
 $EndComp
 $Comp
@@
 F 3 "" H 7725 4300 50  0000 C CNN
 	1    7725 4300
-	-1   0    0    -1
+	-1   0    0    1
 $EndComp
 $Comp
@@
 Text Label 6600 4450 0    60   ~ 0
 3V3
-Text Label 6600 4350 0    60   ~ 0
+Text Label 7700 3000 0    60   ~ 0
 5V
 Text Label 8050 4350 0    60   ~ 0
@@
 Text Label 10750 1600 0    60   ~ 0
 5V
+Text Label 6600 4350 0    60   ~ 0
+A5(SCL)
 Text Label 6600 4250 0    60   ~ 0
-A5(SCL)
-Text Label 6600 4150 0    60   ~ 0
 A4(SDA)
 Text Label 6600 4050 0    60   ~ 0
@@
 NoConn ~ 9275 1900
 NoConn ~ 10350 2500
-NoConn ~ 10350 2300
 NoConn ~ 10350 2200
 NoConn ~ 10350 2100
@@
 Text Label 10250 3975 0    60   ~ 0
 12(MISO)
+Text Label 10750 2300 0    60   ~ 0
+A1
+Wire Wire Line
+	10350 2300 10750 2300
+Text Label 6600 4150 0    60   ~ 0
+A1
+$Comp
+L CONN_01X02 P10
+U 1 1 57169F53
+P 7350 3050
+F 0 "P10" H 7350 3200 50  0000 C CNN
+F 1 "CONN_01X02" V 7450 3050 50  0000 C CNN
+F 2 "Socket_Strips:Socket_Strip_Straight_1x02" H 7350 3050 50  0001 C CNN
+F 3 "" H 7350 3050 50  0000 C CNN
+	1    7350 3050
+	-1   0    0    1
+$EndComp
+$Comp
+L GND #PWR09
+U 1 1 5716A32E
+P 7550 3100
+F 0 "#PWR09" H 7550 2850 50  0001 C CNN
+F 1 "GND" H 7550 2950 50  0000 C CNN
+F 2 "" H 7550 3100 50  0000 C CNN
+F 3 "" H 7550 3100 50  0000 C CNN
+	1    7550 3100
+	1    0    0    -1
+$EndComp
+Wire Wire Line
+	7550 3000 7700 3000
 $EndSCHEMATC
