File: kicad/nrf_nano/nrf_nano.kicad_pcb (KiCad board)
At the start: 2 copper layers, 50 x 50 mm, 15 parts, among them P1 5V_OUT, P2 ALT_PWR, P3 NRF_24L01, P4 CONN_01X15, P5 CONN_01X06, P6 CONN_01X15, P7 CONN_01X06

Commit message: Switches
Parts:
- added P10: MOUNT_HOLE, Mounting_Holes:MountingHole_3.2mm_M3_Pad, F.Cu at (186.0, 126.0)
- added P11: MOUNT_HOLE, Mounting_Holes:MountingHole_3.2mm_M3_Pad, F.Cu at (144.0, 126.0)
- added P8: MOUNT_HOLE, Mounting_Holes:MountingHole_3.2mm_M3_Pad, F.Cu at (144.0, 84.0)
- added P9: MOUNT_HOLE, Mounting_Holes:MountingHole_3.2mm_M3_Pad, F.Cu at (186.0, 84.0)
- added SW1: SW_PUSH, Buttons_Switches_ThroughHole:SW_PUSH_SMALL, F.Cu at (147.2, 115.2)
- added SW2: SW_PUSH, Buttons_Switches_ThroughHole:SW_PUSH_SMALL, F.Cu at (182.8, 115.2)
- moved D3 38.9 mm to (163.1, 121.5)
- moved P2 36.8 mm to (179.0, 82.1), turned to 270 degrees
- moved R3 22.5 mm to (165.0, 116.4)
- moved D1 21.7 mm to (151.0, 88.5), turned to 270 degrees
- moved D2 21.6 mm to (179.0, 88.5), turned to 270 degrees
- moved R1 21.6 mm to (161.2, 116.4)
- moved R2 21.6 mm to (168.8, 116.4)
- moved R5 12.8 mm to (177.7, 96.1), turned to 270 degrees
- moved R4 8.98 mm to (148.5, 107.5)
- moved P1 3.81 mm to (153.6, 82.1), turned to 180 degrees
- moved P3 3.81 mm to (165.0, 98.7)
