File: kicad/nrf_nano/nrf_nano.sch (KiCad schematic (older format))
At the start: 15 parts, among them P1 5V_OUT, P2 ALT_PWR, P3 NRF_24L01, P4 CONN_01X15, P5 CONN_01X06, P6 CONN_01X15, P7 CONN_01X06

Commit message: Switches
Parts:
- added P10, P11, P8, P9: MOUNT_HOLE, Mounting_Holes:MountingHole_3.2mm_M3_Pad, symbol CONN_01X01
- added SW1, SW2: SW_PUSH, Buttons_Switches_ThroughHole:SW_PUSH_SMALL, symbol SW_PUSH
Connections:
- net D2: now also SW1.2
- net D7: now also SW2.2
- net GND: now also P10.1 (P1), P11.1 (P1), P8.1 (P1), P9.1 (P1), SW1.1, SW2.1
Changed lines of the file:
@@
 LIBS:contrib
 LIBS:valves
+LIBS:nrf_nano-cache
 EELAYER 25 0
 EELAYER END
@@
 VIN
 $Comp
-L GND #PWR01
+L GND #PWR16
 U 1 1 57177355
 P 10600 1050
-F 0 "#PWR01" H 10600 800 50  0001 C CNN
+F 0 "#PWR16" H 10600 800 50  0001 C CNN
 F 1 "GND" H 10600 900 50  0000 C CNN
 F 2 "" H 10600 1050 50  0000 C CNN
@@
 D3
 $Comp
-L GND #PWR02
+L GND #PWR13
 U 1 1 571773E2
 P 8500 1250
-F 0 "#PWR02" H 8500 1000 50  0001 C CNN
+F 0 "#PWR13" H 8500 1000 50  0001 C CNN
 F 1 "GND" H 8500 1100 50  0000 C CNN
 F 2 "" H 8500 1250 50  0000 C CNN
@@
 LED_GREEN
 $Comp
-L GND #PWR03
+L GND #PWR7
 U 1 1 571776E2
 P 6050 1850
-F 0 "#PWR03" H 6050 1600 50  0001 C CNN
+F 0 "#PWR7" H 6050 1600 50  0001 C CNN
 F 1 "GND" H 6050 1700 50  0000 C CNN
 F 2 "" H 6050 1850 50  0000 C CNN
@@
 $EndComp
 $Comp
-L GND #PWR04
+L GND #PWR8
 U 1 1 571776FF
 P 6050 2350
-F 0 "#PWR04" H 6050 2100 50  0001 C CNN
+F 0 "#PWR8" H 6050 2100 50  0001 C CNN
 F 1 "GND" H 6050 2200 50  0000 C CNN
 F 2 "" H 6050 2350 50  0000 C CNN
@@
 $EndComp
 $Comp
-L GND #PWR05
+L GND #PWR9
 U 1 1 5717781B
 P 6150 3150
-F 0 "#PWR05" H 6150 2900 50  0001 C CNN
+F 0 "#PWR9" H 6150 2900 50  0001 C CNN
 F 1 "GND" H 6150 3000 50  0000 C CNN
 F 2 "" H 6150 3150 50  0000 C CNN
@@
 3V3
 $Comp
-L GND #PWR06
+L GND #PWR12
 U 1 1 57177C2F
 P 7600 3800
-F 0 "#PWR06" H 7600 3550 50  0001 C CNN
+F 0 "#PWR12" H 7600 3550 50  0001 C CNN
 F 1 "GND" H 7600 3650 50  0000 C CNN
 F 2 "" H 7600 3800 50  0000 C CNN
@@
 VIN
 $Comp
-L GND #PWR07
+L GND #PWR10
 U 1 1 57177E5B
 P 7350 2200
-F 0 "#PWR07" H 7350 1950 50  0001 C CNN
+F 0 "#PWR10" H 7350 1950 50  0001 C CNN
 F 1 "GND" H 7350 2050 50  0000 C CNN
 F 2 "" H 7350 2200 50  0000 C CNN
@@
 5V
 $Comp
-L GND #PWR08
+L GND #PWR11
 U 1 1 57178072
 P 7450 2800
-F 0 "#PWR08" H 7450 2550 50  0001 C CNN
+F 0 "#PWR11" H 7450 2550 50  0001 C CNN
 F 1 "GND" H 7450 2650 50  0000 C CNN
 F 2 "" H 7450 2800 50  0000 C CNN
@@
 $EndComp
 $Comp
-L GND #PWR09
+L GND #PWR14
 U 1 1 5717841B
 P 9350 4150
-F 0 "#PWR09" H 9350 3900 50  0001 C CNN
+F 0 "#PWR14" H 9350 3900 50  0001 C CNN
 F 1 "GND" H 9350 4000 50  0000 C CNN
 F 2 "" H 9350 4150 50  0000 C CNN
@@
 $EndComp
 $Comp
-L GND #PWR010
+L GND #PWR15
 U 1 1 57178453
 P 10450 4150
-F 0 "#PWR010" H 10450 3900 50  0001 C CNN
+F 0 "#PWR15" H 10450 3900 50  0001 C CNN
 F 1 "GND" H 10450 4000 50  0000 C CNN
 F 2 "" H 10450 4150 50  0000 C CNN
@@
 Text GLabel 10450 3650 2    60   Input ~ 0
 SS
+$Comp
+L SW_PUSH SW1
+U 1 1 57178D5C
+P 5100 4350
+F 0 "SW1" H 5250 4460 50  0000 C CNN
+F 1 "SW_PUSH" H 5100 4270 50  0000 C CNN
+F 2 "Buttons_Switches_ThroughHole:SW_PUSH_SMALL" H 5100 4350 50  0001 C CNN
+F 3 "" H 5100 4350 50  0000 C CNN
+	1    5100 4350
+	1    0    0    -1
+$EndComp
+$Comp
+L SW_PUSH SW2
+U 1 1 57178D9F
+P 5100 4850
+F 0 "SW2" H 5250 4960 50  0000 C CNN
+F 1 "SW_PUSH" H 5100 4770 50  0000 C CNN
+F 2 "Buttons_Switches_ThroughHole:SW_PUSH_SMALL" H 5100 4850 50  0001 C CNN
+F 3 "" H 5100 4850 50  0000 C CNN
+	1    5100 4850
+	1    0    0    -1
+$EndComp
+Text GLabel 5400 4350 2    60   Input ~ 0
+D2
+Text GLabel 5400 4850 2    60   Input ~ 0
+D7
+$Comp
+L GND #PWR5
+U 1 1 57178F4E
+P 4800 4350
+F 0 "#PWR5" H 4800 4100 50  0001 C CNN
+F 1 "GND" H 4800 4200 50  0000 C CNN
+F 2 "" H 4800 4350 50  0000 C CNN
+F 3 "" H 4800 4350 50  0000 C CNN
+	1    4800 4350
+	1    0    0    -1
+$EndComp
+$Comp
+L GND #PWR6
+U 1 1 57178F8C
+P 4800 4850
+F 0 "#PWR6" H 4800 4600 50  0001 C CNN
+F 1 "GND" H 4800 4700 50  0000 C CNN
+F 2 "" H 4800 4850 50  0000 C CNN
+F 3 "" H 4800 4850 50  0000 C CNN
+	1    4800 4850
+	1    0    0    -1
+$EndComp
+$Comp
+L CONN_01X01 P8
+U 1 1 5717927C
+P 2200 1450
+F 0 "P8" H 2200 1550 50  0000 C CNN
+F 1 "MOUNT_HOLE" V 2300 1450 50  0000 C CNN
+F 2 "Mounting_Holes:MountingHole_3.2mm_M3_Pad" H 2200 1450 50  0001 C CNN
+F 3 "" H 2200 1450 50  0000 C CNN
+	1    2200 1450
+	0    -1   -1   0
+$EndComp
+$Comp
+L CONN_01X01 P10
+U 1 1 57179324
+P 2800 1450
+F 0 "P10" H 2800 1550 50  0000 C CNN
+F 1 "MOUNT_HOLE" V 2900 1450 50  0000 C CNN
+F 2 "Mounting_Holes:MountingHole_3.2mm_M3_Pad" H 2800 1450 50  0001 C CNN
+F 3 "" H 2800 1450 50  0000 C CNN
+	1    2800 1450
+	0    -1   -1   0
+$EndComp
+$Comp
+L CONN_01X01 P9
+U 1 1 57179385
+P 2200 2150
+F 0 "P9" H 2200 2250 50  0000 C CNN
+F 1 "MOUNT_HOLE" V 2300 2150 50  0000 C CNN
+F 2 "Mounting_Holes:MountingHole_3.2mm_M3_Pad" H 2200 2150 50  0001 C CNN
+F 3 "" H 2200 2150 50  0000 C CNN
+	1    2200 2150
+	0    -1   -1   0
+$EndComp
+$Comp
+L CONN_01X01 P11
+U 1 1 57179413
+P 2800 2150
+F 0 "P11" H 2800 2250 50  0000 C CNN
+F 1 "MOUNT_HOLE" V 2900 2150 50  0000 C CNN
+F 2 "Mounting_Holes:MountingHole_3.2mm_M3_Pad" H 2800 2150 50  0001 C CNN
+F 3 "" H 2800 2150 50  0000 C CNN
+	1    2800 2150
+	0    -1   -1   0
+$EndComp
+$Comp
+L GND #PWR1
+U 1 1 57179482
+P 2200 1650
+F 0 "#PWR1" H 2200 1400 50  0001 C CNN
+F 1 "GND" H 2200 1500 50  0000 C CNN
+F 2 "" H 2200 1650 50  0000 C CNN
+F 3 "" H 2200 1650 50  0000 C CNN
+	1    2200 1650
+	1    0    0    -1
+$EndComp
+$Comp
+L GND #PWR3
+U 1 1 57179569
+P 2800 1650
+F 0 "#PWR3" H 2800 1400 50  0001 C CNN
+F 1 "GND" H 2800 1500 50  0000 C CNN
+F 2 "" H 2800 1650 50  0000 C CNN
+F 3 "" H 2800 1650 50  0000 C CNN
+	1    2800 1650
+	1    0    0    -1
+$EndComp
+$Comp
+L GND #PWR4
+U 1 1 571795B3
+P 2800 2350
+F 0 "#PWR4" H 2800 2100 50  0001 C CNN
+F 1 "GND" H 2800 2200 50  0000 C CNN
+F 2 "" H 2800 2350 50  0000 C CNN
+F 3 "" H 2800 2350 50  0000 C CNN
+	1    2800 2350
+	1    0    0    -1
+$EndComp
+$Comp
+L GND #PWR2
+U 1 1 5717963C
+P 2200 2350
+F 0 "#PWR2" H 2200 2100 50  0001 C CNN
+F 1 "GND" H 2200 2200 50  0000 C CNN
+F 2 "" H 2200 2350 50  0000 C CNN
+F 3 "" H 2200 2350 50  0000 C CNN
+	1    2200 2350
+	1    0    0    -1
+$EndComp
 $EndSCHEMATC
